Commit message: [Update]Change wheel hardware interface to Effort

File: swerve_drive_robot_description/robot/swerve_drive_robot.urdf.xacro (robot description, xacro)
@@ -62,5 +62,5 @@
 			<robotNamespace>/swerve_drive_robot/wheel</robotNamespace>
 			<robotSimType>gazebo_ros_control/DefaultRobotHWSim</robotSimType>
-			<legacyModeNS>false</legacyModeNS>
+			<legacyModeNS>true</legacyModeNS>
 		</plugin>
 	</gazebo>
@@ -69,5 +69,5 @@
 			<robotNamespace>/swerve_drive_robot/steering</robotNamespace>
 			<robotSimType>gazebo_ros_control/DefaultRobotHWSim</robotSimType>
-			<legacyModeNS>false</legacyModeNS>
+			<legacyModeNS>true</legacyModeNS>
 		</plugin>
 	</gazebo>

File: swerve_drive_robot_description/urdf/swerve_drive/steering.transmission.xacro (robot description, xacro)
@@ -8,5 +8,4 @@
             </joint>
             <actuator name="${prefix}_steering_motor">
-                <hardwareInterface>hardware_interface/VelocityJointInterface</hardwareInterface>
                 <mechanicalReduction>1</mechanicalReduction>
             </actuator>

File: swerve_drive_robot_description/urdf/swerve_drive/swerve_drive.gazebo.xacro (robot description, xacro)
@@ -5,6 +5,6 @@
         <gazebo reference="${prefix}_steering_link">
             <selfCollide>false</selfCollide>
-            <mu1 value="0.8" />
-            <mu2 value="0.8" />
+            <mu1 value="0.4" />
+            <mu2 value="0.4" />
             <kp>1e8</kp>
             <kd>1e8</kd>
@@ -13,6 +13,6 @@
         <gazebo reference="${prefix}_wheel_link">
             <selfCollide>false</selfCollide>
-            <mu1 value="0.8" />
-            <mu2 value="0.8" />
+            <mu1 value="0.4" />
+            <mu2 value="0.4" />
             <kp>1e8</kp>
             <kd>1e8</kd>

File: swerve_drive_robot_description/urdf/swerve_drive/swerve_drive.urdf.xacro (robot description, xacro)
@@ -18,5 +18,5 @@
             <child link="${prefix}_steering_link"/>
             <xacro:insert_block name="joint_axis_s"/>
-            <limit lower="-${M_PI}" upper="${M_PI}" effort="100" velocity="100"/>
+            <limit lower="-${M_PI}" upper="${M_PI}" effort="10" velocity="10"/>
         </joint>
         <link name="${prefix}_steering_link">
@@ -45,6 +45,6 @@
             <child link="${prefix}_wheel_link"/>
             <xacro:insert_block name="joint_axis_w"/>
-            <limit velocity="12.0" effort="10" />
-            <dynamics damping="0.01"/>
+            <limit velocity="15.0" effort="0.001" />
+            <dynamics damping="0"/>
         </joint>
         <link name="${prefix}_wheel_link">

File: swerve_drive_robot_description/urdf/swerve_drive/wheel.transmission.xacro (robot description, xacro)
@@ -5,8 +5,7 @@
             <type>transmission_interface/SimpleTransmission</type>
             <joint name="${prefix}_wheel_joint">
-                <hardwareInterface>hardware_interface/VelocityJointInterface</hardwareInterface>
+                <hardwareInterface>hardware_interface/EffortJointInterface</hardwareInterface>
             </joint>
             <actuator name="${prefix}_wheel_motor">
-                <hardwareInterface>hardware_interface/VelocityJointInterface</hardwareInterface>
                 <mechanicalReduction>1</mechanicalReduction>
             </actuator>
